Commit message: update urdf

File: pyroki_ik/URDF/gripper/d1_description/urdf/d1_description.urdf (robot description, URDF)
Before this commit: robot d1_description, 10 links, 9 joints
Links:
- link Link1: geometry collision mesh filename=../meshes/Link1.STL; visual mesh filename=../meshes/Link1.STL
- link Link2: geometry collision mesh filename=../meshes/Link2.STL; visual mesh filename=../meshes/Link2.STL
- link Link3: geometry collision mesh filename=../meshes/Link3.STL; visual mesh filename=../meshes/Link3.STL
- link Link4: geometry collision mesh filename=../meshes/Link4.STL; visual mesh filename=../meshes/Link4.STL
- link Link5: geometry collision mesh filename=../meshes/Link5.STL; visual mesh filename=../meshes/Link5.STL
- link Link6: geometry collision mesh filename=../meshes/Link6.STL; visual mesh filename=../meshes/Link6.STL
- link Link7_1: geometry collision mesh filename=../meshes/Link7_1.STL; visual mesh filename=../meshes/Link7_1.STL
- link Link7_2: geometry collision mesh filename=../meshes/Link7_2.STL; visual mesh filename=../meshes/Link7_2.STL
- link Link_tcp: geometry collision mesh filename=../meshes/Link7_2.STL; visual mesh filename=../meshes/Link7_2.STL
- link base_link: geometry collision mesh filename=../meshes/base_link.STL; visual mesh filename=../meshes/base_link.STL
