Commit message: update assets

File: assets/urdf/d1_description_1.urdf (robot description, URDF)
Before this commit: robot d1_description, 9 links, 8 joints
Joints:
- joint Joint1: axis 0 0 -1 -> 0 0 1
- joint Joint4: axis 0 0 -1 -> 0 0 1
- joint Joint7_1: limit lower=-0.03 upper=0.03 effort=0 velocity=0 -> lower=0 upper=0.03 effort=0 velocity=0; origin xyz=-0.0056012 -0.049636 0.0706 rpy=-1.5714 -1.5708 0 -> xyz=-0.0056012 -0.029636 0.0706 rpy=-1.5714 -1.5708 0
- joint Joint7_2: limit lower=-0.03 upper=0.03 effort=0 velocity=0 -> lower=-0.03 upper=0 effort=0 velocity=0; mimic joint=Joint7_1 multiplier=-1 offset=0 -> (none); origin xyz=-0.0056388 0.04964 0.0706 rpy=1.5702 -1.5708 0 -> xyz=-0.0056388 0.02964 0.0706 rpy=1.5702 -1.5708 0

File: assets/urdf/d1_description_2.urdf (robot description, URDF)
Before this commit: robot d1_description, 9 links, 8 joints
Links:
- added link Link8, mass 0.001; collision box size=0.002 0.002 0.002; visual box size=0.002 0.002 0.002
Joints:
- added joint Joint8: type fixed, parent Link6, child Link8, origin xyz=0 0 0.11 rpy=0 0 0
- joint Joint6: origin xyz=0.0825 -0.0010782 -0.023822 rpy=-1.5708 0 -1.5708 -> xyz=0.0825 -0.0010782 -0.023822 rpy=-1.5708 -1.5708 -1.5708
